Commit message: prueba de lidar en gazebo

File: urfi_description/urdf/include/common_macros_robot.urdf.xacro (robot description, xacro)
@@ -27,5 +27,5 @@
                 <origin xyz="0 ${reflect * length} 0" rpy="${-1 * reflect * pi/2} 0 0"/>
                 <geometry>
-                    <mesh filename="file:///home/alexoberco/Escritorio/ros2_ws/src/urfi_project/urfi_description/meshes/wheel.stl" scale="${length} ${length} ${length}"/>
+                    <mesh filename="file:///home/rosuser/ws/src/urfi_project/urfi_description/meshes/wheel.stl" scale="${length} ${length} ${length}"/>
                 </geometry>
                 <material name="dark_grey"/>

File: urfi_description/urdf/include/material.urdf.xacro (robot description, xacro)
@@ -25,3 +25,6 @@
     <color rgba="0.3 0.3 0.3 1"/>
   </material>
+  <material name="green">
+    <color rgba="0.0 1.0 0.0 1.0"/>
+  </material>
 </robot>

File: urfi_description/urdf/robot_model.urdf (robot description, URDF)
Before this commit: robot robot_model, 8 links, 7 joints
Links:
- added link base_lidar, mass 4.0; collision box size=0.1 0.3 0.1; visual box size=0.3 0.1 0.1
- link left_1_wheel: geometry collision cylinder length=0.075 radius=0.1; visual mesh filename=file:///home/rosuser/ws/src/urfi_project/urfi_description/m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 scale=0.075 0.075 0.075
- link left_2_wheel: geometry collision cylinder length=0.075 radius=0.1; visual mesh filename=file:///home/rosuser/ws/src/urfi_project/urfi_description/m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 scale=0.075 0.075 0.075
- link left_3_wheel: geometry collision cylinder length=0.075 radius=0.1; visual mesh filename=file:///home/rosuser/ws/src/urfi_project/urfi_description/m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 scale=0.075 0.075 0.075
- link right_1_wheel: geometry collision cylinder length=0.075 radius=0.1; visual mesh filename=file:///home/rosuser/ws/src/urfi_project/urfi_description/m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 scale=0.075 0.075 0.075
- link right_2_wheel: geometry collision cylinder length=0.075 radius=0.1; visual mesh filename=file:///home/rosuser/ws/src/urfi_project/urfi_description/m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 scale=0.075 0.075 0.075
- link right_3_wheel: geometry collision cylinder length=0.075 radius=0.1; visual mesh filename=file:///home/rosuser/ws/src/urfi_project/urfi_description/m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 scale=0.075 0.075 0.075
Joints:
- added joint base_lidar_joint: type fixed, parent base_link, child base_lidar, origin xyz=0.0 0.0 0.0 rpy=0.0 0.0 0.0

File: urfi_description/urdf/robot_model.xacro.urdf (robot description, URDF)
Before this commit: robot robot_model, 1 links, 1 joints
Links:
- added link lidar_link; collision cylinder length=0.0258 radius=0.03185; visual cylinder length=0.0258 radius=0.03185
Joints:
- added joint base_lidar_joint: type fixed, parent base_link, child base_lidar_link, origin xyz=0.0 0.0 0.1 rpy=0.0 0.0 0.0
- added joint lidar_joint: type fixed, parent base_lidar_link, child lidar_link, origin xyz=0.0 0.0 0.05 rpy=0.0 0.0 0.0

Commit message: lidar funcional en ignition y rviz

File: urfi_description/urdf/include/common_macros_robot.urdf.xacro (robot description, xacro)
@@ -27,5 +27,5 @@
                 <origin xyz="0 ${reflect * length} 0" rpy="${-1 * reflect * pi/2} 0 0"/>
                 <geometry>
-                    <mesh filename="file:///home/rosuser/ws/src/urfi_project/urfi_description/meshes/wheel.stl" scale="${length} ${length} ${length}"/>
+                    <mesh filename="file:///home/alexoberco/Escritorio/ros2_ws/src/urfi_project/urfi_description/meshes/wheel.stl" scale="${length} ${length} ${length}"/>
                 </geometry>
                 <material name="dark_grey"/>

File: urfi_description/urdf/robot_model.urdf (robot description, URDF)
Before this commit: robot robot_model, 9 links, 8 joints
Links:
- link right_1_wheel: geometry collision cylinder length=0.075 radius=0.1; visual mesh filename=file:///src/urfi_project/urfi_description/meshes/wheel.stl scale=0.075 0.075 0.075

Commit message: bridge incluido en launch y slam config aniadida

File: urfi_description/urdf/include/common_macros_robot.urdf.xacro (robot description, xacro)
@@ -27,5 +27,5 @@
                 <origin xyz="0 ${reflect * length} 0" rpy="${-1 * reflect * pi/2} 0 0"/>
                 <geometry>
-                    <mesh filename="file:///home/alexoberco/Escritorio/ros2_ws/src/urfi_project/urfi_description/meshes/wheel.stl" scale="${length} ${length} ${length}"/>
+                    <mesh filename="file:///home/alexoberco/Desktop/ros2_ws/src/urfi_project/urfi_description/meshes/wheel.stl" scale="${length} ${length} ${length}"/>
                 </geometry>
                 <material name="dark_grey"/>

Commit message: slam y mapa funcional

File: urfi_description/urdf/include/common_macros_robot.urdf.xacro (robot description, xacro)
@@ -27,5 +27,5 @@
                 <origin xyz="0 ${reflect * length} 0" rpy="${-1 * reflect * pi/2} 0 0"/>
                 <geometry>
-                    <mesh filename="file:///home/alexoberco/Desktop/ros2_ws/src/urfi_project/urfi_description/meshes/wheel.stl" scale="${length} ${length} ${length}"/>
+                    <mesh filename="file:///home/ieeerasjaveriana/Escritorio/alejo_ws/src/urfi_project/urfi_description/meshes/wheel.stl" scale="${length} ${length} ${length}"/>
                 </geometry>
                 <material name="dark_grey"/>

Commit message: mapita improvisado aniadido y launch control y slam arreglados

File: urfi_description/urdf/include/common_macros_robot.urdf.xacro (robot description, xacro)
@@ -27,5 +27,5 @@
                 <origin xyz="0 ${reflect * length} 0" rpy="${-1 * reflect * pi/2} 0 0"/>
                 <geometry>
-                    <mesh filename="file:///home/ieeerasjaveriana/Escritorio/alejo_ws/src/urfi_project/urfi_description/meshes/wheel.stl" scale="${length} ${length} ${length}"/>
+                    <mesh filename="file:///home/alexoberco/Desktop/ros2_ws/src/urfi_project/urfi_description/meshes/wheel.stl" scale="${length} ${length} ${length}"/>
                 </geometry>
                 <material name="dark_grey"/>
